File: hardware/kicad/BarSync/BarSync.kicad_pcb (KiCad board)
At the start: 2 copper layers, 95 x 60 mm, 20 parts, among them J1 MIDI-IN, J2 MIDI-THRU, J3 TimeSig, J4 Divisor, J5 Reset, J6 Connector, U1 6N139, U2 SN7406N

Commit message: Firmware V1.2
Parts:
- J3: value TimeSig -> Custom
Other:
- board text added: "BarSync - MIDI Clock Bar Counter & Visualizer V1.2"
- board text removed: "BarSync - MIDI Clock Bar Counter & Visualizer"

Commit message: FIrmware 1.2
Parts:
- J1: value MIDI-IN -> MIDI:
- J2: value MIDI-THRU -> THRU
- J4: value Divisor -> Grid (Divisor)
Other:
- board text added: "1"
- board text added: "3"
- board text added: "IN 4 5"
Changed lines of the file:
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@@
 		(tags "Through hole pin header THT 1x02 2.54mm single row")
 		(property "Reference" "J1"
-			(at 2.63 -0.27 180)
-			(layer "F.SilkS")
-			(effects
-				(font
-					(size 1 1)
-					(thickness 0.15)
-				)
-			)
-		)
-		(property "Value" "MIDI-IN"
-			(at -0.12 5.73 90)
+			(at 2.63 -1.77 180)
+			(layer "F.SilkS")
+			(effects
+				(font
+					(size 1 1)
+					(thickness 0.15)
+				)
+			)
+		)
+		(property "Value" "MIDI: "
+			(at -2.62 -4.27 180)
 			(layer "F.SilkS")
 			(effects
@@
 			)
 		)
-		(property "Value" "Divisor"
+		(property "Value" "Grid (Divisor)"
 			(at 0 6.04 0)
 			(layer "F.SilkS")
@@
 		(tags "Through hole pin header THT 1x03 2.54mm single row")
 		(property "Reference" "J2"
-			(at 2.63 -0.23 180)
-			(layer "F.SilkS")
-			(effects
-				(font
-					(size 1 1)
-					(thickness 0.15)
-				)
-			)
-		)
-		(property "Value" "MIDI-THRU"
-			(at 0.13 8.02 90)
+			(at 2.63 -1.73 180)
+			(layer "F.SilkS")
+			(effects
+				(font
+					(size 1 1)
+					(thickness 0.15)
+				)
+			)
+		)
+		(property "Value" "THRU"
+			(at -2.62 -2.73 180)
 			(layer "F.SilkS")
 			(effects
@@
 		)
 	)
-	(gr_text "4"
-		(at 97.75 91.25 0)
+	(gr_text "1"
+		(at 98.25 85.75 0)
 		(layer "F.SilkS")
 		(effects
@@
 		)
 	)
-	(gr_text "5"
-		(at 100.5 91.25 0)
+	(gr_text "2\n"
+		(at 101.5 85.75 0)
 		(layer "F.SilkS")
 		(effects
@@
 		)
 	)
-	(gr_text "2"
-		(at 107.75 91.25 0)
+	(gr_text "1"
+		(at 110.25 85.75 0)
 		(layer "F.SilkS")
 		(effects
@@
 		)
 	)
+	(gr_text "2"
+		(at 110.25 91 0)
+		(layer "F.SilkS")
+		(effects
+			(font
+				(size 1 1)
+				(thickness 0.15)
+			)
+			(justify left bottom)
+		)
+	)
+	(gr_text "2"
+		(at 112.75 85.75 0)
+		(layer "F.SilkS")
+		(effects
+			(font
+				(size 1 1)
+				(thickness 0.15)
+			)
+			(justify left bottom)
+		)
+	)
 	(gr_text "4"
-		(at 111.5 91.25 0)
+		(at 112.75 91 0)
 		(layer "F.SilkS")
 		(effects
@@
 		)
 	)
-	(gr_text "5"
-		(at 114.25 91.25 0)
+	(gr_text "3"
+		(at 115.5 85.75 0)
 		(layer "F.SilkS")
 		(effects
@@
 		)
 	)
+	(gr_text "5"
+		(at 115.5 91 0)
+		(layer "F.SilkS")
+		(effects
+			(font
+				(size 1 1)
+				(thickness 0.15)
+			)
+			(justify left bottom)
+		)
+	)
+	(gr_text "IN 4   5"
+		(at 99.25 90.5 0)
+		(layer "F.SilkS")
+		(effects
+			(font
+				(size 1 1)
+				(thickness 0.15)
+			)
+		)
+	)

Commit message: Hardware V1.2
Parts:
- J1: value MIDI: -> MIDI
- moved R1 9.89 mm to (82.0, 87.8), turned to 90 degrees
- moved D1 7.19 mm to (88.2, 77.7)
Connections:
- J1 pad 2: Net-(J1-Pin_2) -> Net-(D1-A)
- R1 pad 2: Net-(D1-A) -> Net-(D1-K)
- U1 pad 3: Net-(J1-Pin_2) -> Net-(D1-A)
Routing:
- net Net-(D1-A): track 5.79 -> 39.2 mm
- net Net-(J1-Pin_2): track 28.6 -> 0.00 mm
- net Net-(J1-Pin_1): track 6.38 -> 16.3 mm
- net Net-(D1-K): track 14.3 -> 23.8 mm
