File: hardware/kicad/BarSync/BarSync.kicad_sch (KiCad schematic)
At the start: 16 parts, among them J1 MIDI-IN, J2 MIDI-THRU, J3 TimeSig Switch, J4 Divisor Switch, J5 Reset Switch, J6 Connector, U1 6N139, U2 SN7406N

Commit message: Firmware V1.2
Parts:
- J3: value TimeSig Switch -> Custom Switch
Changed lines of the file:
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@@
 	(title_block
 		(title "BarSync - MIDI Clock Bar Counter & Visualizer")
-		(date "2026-08-21")
-		(rev "1.1")
+		(date "2026-09-02")
+		(rev "1.2")
 	)
 	(arc
@@
 			)
 		)
-		(property "Value" "TimeSig Switch"
+		(property "Value" "Custom Switch"
 			(at 241.046 112.522 0)
 			(show_name no)

Commit message: FIrmware 1.2
Parts:
- J4: value Divisor Switch -> Grid (Divisor) Switch
Changed lines of the file:
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@@
 			)
 		)
-		(property "Value" "Divisor Switch"
+		(property "Value" "Grid (Divisor) Switch"
 			(at 241.808 102.616 0)
 			(show_name no)

Commit message: Hardware V1.2
Parts:
- J2: value MIDI-THRU -> MIDI-THRU 1
Connections:
- net at J1.2 (Pin_2), U1.3: now also D1.2 (A)
- net at R1.2: now also D1.1 (K), U1.2; no longer D1.2 (A)
Other:
- moved on the sheet: R1
